File: PCBussinesCard_Circuit/PCBussinesCard.kicad_sch (KiCad schematic)
At the start: 0 parts

Commit message: Schematic and layout sketch
Parts:
- added C1, C2, C3, C4: 100nF, Capacitor_SMD:C_0402_1005Metric, symbol Device:C_Small
- added C5: 10nF, Capacitor_SMD:C_0402_1005Metric, symbol Device:C_Small
- added C6: 1uF, Capacitor_SMD:C_0402_1005Metric, symbol Device:C_Small
- added D1: RCLAMP0582B, Package_TO_SOT_SMD:SOT-416, symbol Power_Protection:RCLAMP0582B
- added J1: Conn_ARM_JTAG_SWD_10, Connector_PinHeader_1.27mm:PinHeader_2x05_P1.27mm_Vertical_SMD, symbol Connector:Conn_ARM_JTAG_SWD_10
- added J2: USB_A_PCB, ProjectLibrary:PCB_USB_A, symbol Project_library:USB_A_PCB
- added J3: Conn_01x13_Pin, Connector_PinHeader_2.54mm:PinHeader_1x13_P2.54mm_Vertical, symbol Connector:Conn_01x13_Pin
- added U1: STM32L552CCTx, Package_QFP:LQFP-48_7x7mm_P0.5mm, symbol MCU_ST_STM32L5:STM32L552CCTx
- added U2: AP7370-33FDC, Package_DFN_QFN:DFN-6-1EP_2x2mm_P0.65mm_EP1.01x1.7mm, symbol Regulator_Linear:AP7370-33FDC
Connections:
- new net +3.3V: C1.1, C2.1, C3.1, C4.1, C5.1, C6.1, J1.1 (VTref), U1.1 (VBAT), U1.24 (VDD), U1.36 (VDD), U1.48 (VDD), U1.9 (VDDA), U2.1 (VO)
- new net +5V: J2.1 (VBUS), U2.6 (VI)
- new net GND: C1.2, C2.2, C3.2, C4.2, C5.2, C6.2, D1.3 (A), J1.3 (GND), J1.5 (GND), J1.9 (GNDDetect), J2.4 (GND), U1.23 (VSS), U1.35 (VSS), U1.47 (VSS), U1.8 (VSSA), U2.3 (GND), U2.7 (GND)
- new net NRST: J1.10 (~{RESET}), U1.7 (NRST)
- new net SWCLK: J1.4 (SWCLK/TCK), U1.37 (PA14)
- new net SWDIO: J1.2 (SWDIO/TMS), U1.34 (PA13)
- new net USB_D+: D1.2 (K2), J2.3 (D+), U1.33 (PA12)
- new net USB_D-: D1.1 (K1), J2.2 (D-), U1.32 (PA11)
- no-connect marks 0 -> 2
