File: PCBussinesCard_Circuit/PCBussinesCard.kicad_pcb (KiCad board)
At the start: 2 copper layers, 85 x 55 mm, 16 parts, among them IC1 NT2H1311F0DTL, J1 Conn_ARM_JTAG_SWD_10, J2 USB_A_PCB, J3 Conn_01x13_Pin, J4 Conn_01x13_Pin, U1 STM32L552CCTx, U2 AP7370-33FDC

Commit message: cleanup and reorganizing
Parts:
- removed J1: Conn_ARM_JTAG_SWD_10, Connector_PinHeader_1.27mm:PinHeader_2x05_P1.27mm_Vertical_SMD
- added G***: LOGO, ProjectLibrary:QrCode, F.Cu at (125.2, 102.3)
- J3, J4: value Conn_01x13_Pin -> Conn_01x12_Socket; footprint Connector_PinHeader_2.54mm:PinHeader_1x13_P2.54mm_Vertical -> Connector_PinHeader_2.54mm:PinHeader_1x12_P2.54mm_Vertical
- moved IC1 11.5 mm to (139.4, 113.5)
- moved C4 8.43 mm to (161.0, 116.1), turned to -45 degrees
- moved C1 7.77 mm to (156.3, 107.8), turned to -135 degrees
- moved C3 7.05 mm to (164.6, 116.1), turned to -135 degrees
- moved C6 6.53 mm to (169.0, 113.4)
- moved C5 6.53 mm to (168.2, 112.8)
- moved U1 6.53 mm to (162.8, 109.7)
- moved D2 5.25 mm to (170.2, 85.1)
- moved R1 5.25 mm to (171.4, 86.3)
- moved U2 5.25 mm to (173.1, 87.8)
- moved C2 5.21 mm to (164.7, 103.3)
- moved J3 4.29 mm to (178.5, 98.2)
- moved D1 3.50 mm to (174.8, 89.8)
- moved J4 3.18 mm to (182.1, 98.2)
Routing:
- net Net-(IC1-LA): track 0.00 -> 714.3 mm, vias 0 -> 2
- net (no net): track 706.3 -> 0.00 mm
- net +3.3V: track 90.6 -> 0.00 mm, vias 2 -> 0
- net /USB_D+: track 34.1 -> 0.00 mm
- net /USB_D-: track 33.6 -> 0.00 mm
- net /NRST: track 21.6 -> 0.00 mm, vias 1 -> 0
- net /SWDIO: track 20.6 -> 0.00 mm, vias 1 -> 0
- net /SWCLK: track 14.2 -> 0.00 mm, vias 1 -> 0
- net +5V: track 9.30 -> 0.00 mm
- net GND: track 4.10 -> 0.00 mm, vias 2 -> 0
- net Net-(D2-A): track 1.71 -> 0.00 mm
Other:
- outline, holes or cut-outs redrawn
- board text added: "... .-. .. .-. .- -.-. .... .-"
- board text added: "Hardware Design | Robotics | Control"
- board text added: "santiagov3lasquez@gmail.com (+57) 300-895-2758"
- board text removed: "github.com/vekkax"
- board text removed: "santiagov3lasquez@gmail.com"

Commit message: Version 1.0
Parts:
- removed J4: Conn_01x12_Socket, Connector_PinHeader_2.54mm:PinHeader_1x12_P2.54mm_Vertical
- added 0201: C_0201_0603Metric, Capacitor_SMD:C_0201_0603Metric, B.Cu at (162.2, 82.8)
- added 0402: R_0402_1005Metric, Resistor_SMD:R_0402_1005Metric, B.Cu at (157.8, 82.8)
- added 0603: R_0603_1608Metric, Resistor_SMD:R_0603_1608Metric, B.Cu at (153.1, 82.8)
- added 0805: R_0805_2012Metric, Resistor_SMD:R_0805_2012Metric, B.Cu at (147.8, 82.8)
- added 1206: R_1206_3216Metric, Resistor_SMD:R_1206_3216Metric, B.Cu at (142.2, 82.8)
- added 1812: R_1812_4532Metric, Resistor_SMD:R_1812_4532Metric, B.Cu at (135.6, 82.8)
- added 2010: R_2010_5025Metric_Pad1.40x2.65mm_HandSolder, Resistor_SMD:R_2010_5025Metric_Pad1.40x2.65mm_HandSolder, B.Cu at (128.5, 82.8)
- added 2512: R_2512_6332Metric, Resistor_SMD:R_2512_6332Metric, B.Cu at (121.5, 82.8)
- added 2816: R_2816_7142Metric, Resistor_SMD:R_2816_7142Metric, B.Cu at (113.5, 82.8)
- added 4020: R_4020_10251Metric, Resistor_SMD:R_4020_10251Metric, B.Cu at (104.6, 82.8)
- added J1: Conn_01x04_Pin, Connector_PinHeader_2.54mm:PinHeader_1x04_P2.54mm_Horizontal, F.Cu at (167.0, 128.0)
- added LQFP-32 0.5: LQFP-32_5x5mm_P0.5mm, Package_QFP:LQFP-32_5x5mm_P0.5mm, B.Cu at (141.2, 122.2)
- added LQFP-32 0.8: LQFP-32_7x7mm_P0.8mm, Package_QFP:LQFP-32_7x7mm_P0.8mm, B.Cu at (128.2, 122.2)
- added QFN-16: QFN-16-1EP_3x3mm_P0.5mm_EP1.7x1.7mm, Package_DFN_QFN:QFN-16-1EP_3x3mm_P0.5mm_EP1.7x1.7mm, B.Cu at (159.8, 122.2)
- added QFN-32 : QFN-32-1EP_4x4mm_P0.4mm_EP2.9x2.9mm, Package_DFN_QFN:QFN-32-1EP_4x4mm_P0.4mm_EP2.9x2.9mm, B.Cu at (151.5, 122.2)
- added SOT-223: SOT-223, Package_TO_SOT_SMD:SOT-223, B.Cu at (150.1, 111.3)
- added SOT-23-3: SOT-23-3, Package_TO_SOT_SMD:SOT-23-3, B.Cu at (145.9, 102.0)
- added SOT-23-5: SOT-23-5, Package_TO_SOT_SMD:SOT-23-5, B.Cu at (154.7, 102.0)
- added TSSOP-16: TSSOP-16-1EP_4.4x5mm_P0.65mm_EP3x3mm, Package_SO:TSSOP-16-1EP_4.4x5mm_P0.65mm_EP3x3mm, B.Cu at (116.7, 122.0)
- added TSSOP-24: TSSOP-24-1EP_4.4x7.8mm_P0.65mm_EP3.2x5mm, Package_SO:TSSOP-24-1EP_4.4x7.8mm_P0.65mm_EP3.2x5mm, B.Cu at (106.2, 122.0)
- J3: value Conn_01x12_Socket -> Conn_02x12_Odd_Even; footprint Connector_PinHeader_2.54mm:PinHeader_1x12_P2.54mm_Vertical -> Connector_PinSocket_2.54mm:PinSocket_2x12_P2.54mm_Vertical
- moved C4 13.9 mm to (156.1, 103.1), turned to -135 degrees
- moved C3 12.4 mm to (156.2, 106.8), turned to 135 degrees
- moved C1 12.3 mm to (164.5, 98.6), turned to 135 degrees
- moved C6 10.7 mm to (159.0, 109.7), turned to 135 degrees
- moved C5 10.2 mm to (158.3, 110.4), turned to 135 degrees
- moved C2 5.69 mm to (169.0, 107.0), turned to 45 degrees
- moved U1 4.63 mm to (162.6, 105.1), turned to 45 degrees
- moved J3 2.82 mm to (181.3, 98.2)
Connections:
- J3 pad 1: unconnected-(J3-Pin_1-Pad1) -> +5V
- J3 pad 10: unconnected-(J3-Pin_10-Pad10) -> /PB1
- J3 pad 11: unconnected-(J3-Pin_11-Pad11) -> /PB14
- J3 pad 12: unconnected-(J3-Pin_12-Pad12) -> /PB0
- J3 pad 2: unconnected-(J3-Pin_2-Pad2) -> +3.3V
- J3 pad 3: unconnected-(J3-Pin_3-Pad3) -> /PA10
- J3 pad 4: unconnected-(J3-Pin_4-Pad4) -> /PB11
- J3 pad 5: unconnected-(J3-Pin_5-Pad5) -> /PA9
- J3 pad 6: unconnected-(J3-Pin_6-Pad6) -> /PB10
- J3 pad 7: unconnected-(J3-Pin_7-Pad7) -> /PA8
- J3 pad 8: unconnected-(J3-Pin_8-Pad8) -> /PB2
- J3 pad 9: unconnected-(J3-Pin_9-Pad9) -> /PB15
- U1 pad 10: unconnected-(U1-PA0-Pad10) -> /PA0
- U1 pad 11: unconnected-(U1-PA1-Pad11) -> /PA1
- U1 pad 12: unconnected-(U1-PA2-Pad12) -> /PA2
- U1 pad 13: unconnected-(U1-PA3-Pad13) -> /PA3
- U1 pad 14: unconnected-(U1-PA4-Pad14) -> /PA4
- U1 pad 15: unconnected-(U1-PA5-Pad15) -> /PA5
- U1 pad 16: unconnected-(U1-PA6-Pad16) -> /PA6
- U1 pad 17: unconnected-(U1-PA7-Pad17) -> /PA7
- U1 pad 18: unconnected-(U1-PB0-Pad18) -> /PB0
- U1 pad 19: unconnected-(U1-PB1-Pad19) -> /PB1
- U1 pad 20: unconnected-(U1-PB2-Pad20) -> /PB2
- U1 pad 21: unconnected-(U1-PB10-Pad21) -> /PB10
- U1 pad 22: unconnected-(U1-PB11-Pad22) -> /PB11
- U1 pad 25: unconnected-(U1-PB12-Pad25) -> /PB12
- U1 pad 26: unconnected-(U1-PB13-Pad26) -> /PB13
- U1 pad 27: unconnected-(U1-PB14-Pad27) -> /PB14
- U1 pad 28: unconnected-(U1-PB15-Pad28) -> /PB15
- U1 pad 29: unconnected-(U1-PA8-Pad29) -> /PA8
- U1 pad 30: unconnected-(U1-PA9-Pad30) -> /PA9
- U1 pad 31: unconnected-(U1-PA10-Pad31) -> /PA10
- U1 pad 38: unconnected-(U1-PA15-Pad38) -> /PA15
- U1 pad 39: unconnected-(U1-PB3-Pad39) -> /PB3
- U1 pad 40: unconnected-(U1-PB4-Pad40) -> /PB4
- U1 pad 41: unconnected-(U1-PB5-Pad41) -> /PB5
- U1 pad 42: unconnected-(U1-PB6-Pad42) -> /PB6
- U1 pad 43: unconnected-(U1-PB7-Pad43) -> /PB7
- U1 pad 45: unconnected-(U1-PB8-Pad45) -> /PB8
- U1 pad 46: unconnected-(U1-PB9-Pad46) -> /PB9
Routing:
- net +3.3V: track 0.00 -> 97.9 mm, vias 0 -> 2
- net /SWDIO: track 0.00 -> 38.6 mm, vias 0 -> 1
- net /SWCLK: track 0.00 -> 38.6 mm, vias 0 -> 1
- net /PA0: track 0.00 -> 30.4 mm, vias 0 -> 1
- net +5V: track 0.00 -> 28.6 mm, vias 0 -> 1
- net /PA1: track 0.00 -> 28.6 mm, vias 0 -> 1
- net (no net): track 0.00 -> 28.1 mm
- net /PA2: track 0.00 -> 27.2 mm, vias 0 -> 1
- net /USB_D-: track 0.00 -> 24.9 mm
- net /USB_D+: track 0.00 -> 24.7 mm
- net /PB12: track 0.00 -> 24.4 mm, vias 0 -> 1
- net /PB13: track 0.00 -> 22.9 mm, vias 0 -> 1
- net /PB14: track 0.00 -> 21.5 mm, vias 0 -> 1
- net /PA3: track 0.00 -> 20.8 mm
- net /PB15: track 0.00 -> 20.8 mm, vias 0 -> 1
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Other:
- board text added: "10"
- board text added: "100"
- board text added: "12"
- board text added: "15"
- board text added: "20"
- board text added: "30"
- board text added: "3V3"
- board text added: "40"
- board text added: "50"
- board text added: "5V"
- board text added: "70"
- board text added: "8"
- board text added: "A1"
- board text added: "A10"
- board text added: "A2"
- board text added: "A3"
- board text added: "A4"
- board text added: "A5"
- board text added: "A6"
- board text added: "A7"
- board text added: "A8"
- board text added: "A9"
- board text added: "AO"
- board text added: "B0"
- board text added: "B1"
- board text added: "B10"
- board text added: "B11"
- board text added: "B12"
- board text added: "B13"
- board text added: "B14"
- board text added: "B15"
- board text added: "B2"
- board text added: "CLK"
- board text added: "Connect the USB to learn more"
- board text added: "GND"
- board text added: "IO"
- board text added: "Learn more about this project and make your own PCBussinesCard at: github.com/vekkax/PCBussinessCard"
- board text added: "SWD"
- board text added: "Tap or Scan"
- board text added: "Trace Width (mil)"
- board text added: "Use me as a Dev Board!"

Commit message: Production V1.0
Parts:
- removed U1: STM32L552CCTx, Package_QFP:LQFP-48_7x7mm_P0.5mm
- added C7: 100nF, Capacitor_SMD:C_0402_1005Metric, F.Cu at (158.0, 107.9)
- added C8: 100nF, Capacitor_SMD:C_0402_1005Metric, F.Cu at (174.7, 89.8)
- added C9: 100nF, Capacitor_SMD:C_0402_1005Metric, F.Cu at (178.2, 93.2)
- added SW1: SMD_4.6x2.8mm_h1.9mm, PCM_SparkFun-Switch:Push_SMD_4.6x2.8mm_h1.9mm, F.Cu at (167.6, 83.2)
- added U3: LM3480-3.3, Package_TO_SOT_SMD:SOT-23, F.Cu at (176.0, 91.7)
- U2: value AP7370-33FDC -> STM32L452CEUx; footprint Package_DFN_QFN:DFN-6-1EP_2x2mm_P0.65mm_EP1.01x1.7mm -> Package_DFN_QFN:QFN-48-1EP_7x7mm_P0.5mm_EP5.6x5.6mm
- moved U2 20.2 mm to (162.7, 105.1)
- moved D1 2.34 mm to (173.1, 88.3)
- moved 0201 2.28 mm to (164.5, 82.8)
- moved 0603 2.28 mm to (155.3, 82.8)
- moved 0805 2.28 mm to (150.1, 82.8)
- moved 2010 2.28 mm to (130.8, 82.8)
- moved 4020 2.28 mm to (106.9, 82.8)
- moved 2512 2.28 mm to (123.8, 82.8)
- moved 2816 2.28 mm to (115.8, 82.8)
- moved 0402 2.28 mm to (160.1, 82.8)
- moved 1206 2.28 mm to (144.5, 82.8)
- moved 1812 2.28 mm to (137.9, 82.8)
- moved J3 1.52 mm to (179.8, 98.2)
- moved C1 1.50 mm to (163.0, 98.7)
- moved C4 1.21 mm to (156.9, 104.0)
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Connections:
- U2 pad 3: GND -> unconnected-(U2-PC14-Pad3)
- U2 pad 6: +5V -> unconnected-(U2-PH1-Pad6)
- U2 pad 7: GND -> /NRST
Routing:
- net /NRST: track 1.24 -> 34.7 mm, vias 1 -> 2
- net /PA2: track 27.2 -> 24.1 mm
- net +3.3V: track 97.9 -> 100.9 mm, vias 2 -> 3
- net /PB15: track 20.8 -> 17.9 mm
- net +5V: track 28.6 -> 25.8 mm, vias 1 -> 2
- net /PB12: track 24.4 -> 21.6 mm
- net /PB14: track 21.5 -> 19.0 mm
- net /PB13: track 22.9 -> 20.4 mm
- net /PA1: track 28.6 -> 26.2 mm
- net /PA0: track 30.4 -> 28.3 mm
- net GND: track 6.15 -> 4.23 mm, vias 2 -> 30
- net /PA8: track 19.2 -> 17.7 mm
- net /PB10: track 15.4 -> 14.1 mm
- net /SWCLK: track 38.6 -> 39.6 mm
- net /PA10: track 18.3 -> 17.4 mm
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
Commit message: README added and unnecesary files removed
Parts:
- renumbered U2 to U1, U3 to U2
Changed lines of the file:
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@@
 	(net 8 "Net-(D2-A)")
 	(net 9 "Net-(IC1-LA)")
-	(net 10 "unconnected-(U2-PC13-Pad2)")
+	(net 10 "unconnected-(U1-PC13-Pad2)")
 	(net 11 "unconnected-(IC1-FD-Pad3)")
-	(net 12 "unconnected-(U2-PC15-Pad4)")
-	(net 13 "unconnected-(U2-PH1-Pad6)")
-	(net 14 "unconnected-(U2-PC14-Pad3)")
-	(net 15 "unconnected-(U2-PH0-Pad5)")
-	(net 16 "unconnected-(U2-PH3-Pad44)")
+	(net 12 "unconnected-(U1-PC15-Pad4)")
+	(net 13 "unconnected-(U1-PH1-Pad6)")
+	(net 14 "unconnected-(U1-PC14-Pad3)")
+	(net 15 "unconnected-(U1-PH0-Pad5)")
+	(net 16 "unconnected-(U1-PH3-Pad44)")
 	(net 17 "+5V")
 	(net 18 "unconnected-(IC1-EP-Pad5)")
@@
 		(descr "SOT, 3 Pin (JEDEC TO-236 Var AB https://www.jedec.org/document_search?search_api_views_fulltext=TO-236), generated with kicad-footprint-generator ipc_gullwing_generator.py")
 		(tags "SOT TO_SOT_SMD")
-		(property "Reference" "U3"
+		(property "Reference" "U2"
 			(at 0 -2.4 45)
 			(layer "F.SilkS")
@@
 		(descr "QFN, 48 Pin (http://www.st.com/resource/en/datasheet/stm32f042k6.pdf#page=94), generated with kicad-footprint-generator ipc_noLead_generator.py")
 		(tags "QFN NoLead ST_UFQFPN48 Analog_CP-48-13 JEDEC_MO-220-WKKD-4")
-		(property "Reference" "U2"
+		(property "Reference" "U1"
 			(at 0 -4.83 45)
 			(layer "F.SilkS")
@@
 			(layers "F.Cu" "F.Mask" "F.Paste")
 			(roundrect_rratio 0.25)
-			(net 10 "unconnected-(U2-PC13-Pad2)")
+			(net 10 "unconnected-(U1-PC13-Pad2)")
 			(pinfunction "PC13")
 			(pintype "bidirectional")
@@
 			(layers "F.Cu" "F.Mask" "F.Paste")
 			(roundrect_rratio 0.25)
-			(net 14 "unconnected-(U2-PC14-Pad3)")
+			(net 14 "unconnected-(U1-PC14-Pad3)")
 			(pinfunction "PC14")
 			(pintype "bidirectional")
@@
 			(layers "F.Cu" "F.Mask" "F.Paste")
 			(roundrect_rratio 0.25)
-			(net 12 "unconnected-(U2-PC15-Pad4)")
+			(net 12 "unconnected-(U1-PC15-Pad4)")
 			(pinfunction "PC15")
 			(pintype "bidirectional")
@@
 			(layers "F.Cu" "F.Mask" "F.Paste")
 			(roundrect_rratio 0.25)
-			(net 15 "unconnected-(U2-PH0-Pad5)")
+			(net 15 "unconnected-(U1-PH0-Pad5)")
 			(pinfunction "PH0")
 			(pintype "bidirectional")
@@
 			(layers "F.Cu" "F.Mask" "F.Paste")
 			(roundrect_rratio 0.25)
-			(net 13 "unconnected-(U2-PH1-Pad6)")
+			(net 13 "unconnected-(U1-PH1-Pad6)")
 			(pinfunction "PH1")
 			(pintype "bidirectional")
@@
 			(layers "F.Cu" "F.Mask" "F.Paste")
 			(roundrect_rratio 0.25)
-			(net 16 "unconnected-(U2-PH3-Pad44)")
+			(net 16 "unconnected-(U1-PH3-Pad44)")
 			(pinfunction "PH3")
 			(pintype "bidirectional")
